File: digital-driver/driver.sch (KiCad schematic (older format))
At the start: 20 parts, among them J1 Conn_01x04, J2 Conn_01x04, J3 Barrel_Jack, J4 Barrel_Jack, J5 Conn_01x04, J6 LDD-1500L, J7 Conn_01x02, U1 ATtiny85-20PU

Commit message: tap-heatsink
Parts:
- renumbered J6 to U2
Changed lines of the file:
@@
 PWM_LED
 $Comp
-L LDD-1500L:LDD-1500L J6
+L LDD-1500L:LDD-1500L U2
 U 1 1 5FD3EABF
 P 1250 3650
-F 0 "J6" H 2150 3915 50  0000 C CNN
+F 0 "U2" H 2150 3915 50  0000 C CNN
 F 1 "LDD-1500L" H 2150 3824 50  0000 C CNN
 F 2 "LDD-1500L:LDD1500L" H 2900 3750 50  0001 L CNN

Commit message: digital driver 1.0.0
Parts:
- PS1: symbol VXO7805-500-M:VXO7805-500-M -> driver-rescue:VXO7805-500-M-VXO7805-500-M
Connections:
- net GND: now also PS1.2 (GND)
Other:
- moved on the sheet: PS1
Changed lines of the file:
@@
 Connection ~ 6200 4500
 $Comp
-L VXO7805-500-M:VXO7805-500-M PS1
+L driver-rescue:VXO7805-500-M-VXO7805-500-M PS1
 U 1 1 60157AFB
 P 6200 4000

Commit message: digital driver revision B
Parts:
- removed PS1: VXO7805-500-M, CONV_VXO7805-500-M, symbol driver-rescue:VXO7805-500-M-VXO7805-500-M
- added PS1: VXO7805-500-M, CONV_VXO7805-500-M, symbol VXO7805-500-M:VXO7805-500-M
Connections:
- net +12V: now also PS1.1 (+VIN)
- net +5V: now also PS1.3 (+VO)
- net GND: now also J1.1 (Pin_1), J2.1 (Pin_1), PS1.2 (GND); no longer J1.4 (Pin_4), J2.4 (Pin_4)
- net SCL: now also J1.4 (Pin_4), J2.4 (Pin_4); no longer J1.1 (Pin_1), J2.1 (Pin_1)
- net SDA: now also J1.3 (Pin_3), J2.3 (Pin_3); no longer J1.2 (Pin_2), J2.2 (Pin_2)
- new net: J1.2 (Pin_2), J2.2 (Pin_2)
Changed lines of the file:
@@
 Sheet 1 1
 Title "Digital Photoreactor Driver"
-Date "2021-01-22"
-Rev "1.0.0"
+Date "2021-03-06"
+Rev "B"
 Comp "University of Wisconsin-Madison"
 Comment1 "Department of Chemistry"
@@
 L Connector_Generic:Conn_01x04 J1
 U 1 1 5FBC8C0C
-P 4600 1300
-F 0 "J1" H 4680 1292 50  0000 L CNN
-F 1 "Conn_01x04" H 4680 1201 50  0000 L CNN
-F 2 "Connector_JST:JST_PH_S4B-PH-K_1x04_P2.00mm_Horizontal" H 4600 1300 50  0001 C CNN
-F 3 "~" H 4600 1300 50  0001 C CNN
-	1    4600 1300
-	-1   0    0    1
+P 4600 1200
+F 0 "J1" H 4680 1192 50  0000 L CNN
+F 1 "Conn_01x04" H 4680 1101 50  0000 L CNN
+F 2 "Connector_JST:JST_PH_S4B-PH-K_1x04_P2.00mm_Horizontal" H 4600 1200 50  0001 C CNN
+F 3 "~" H 4600 1200 50  0001 C CNN
+	1    4600 1200
+	-1   0    0    -1
 $EndComp
 Text GLabel 6000 1900 2    50   Input ~ 0
@@
 L Connector_Generic:Conn_01x04 J2
 U 1 1 5FE1AA2F
-P 4600 1800
-F 0 "J2" H 4680 1792 50  0000 L CNN
-F 1 "Conn_01x04" H 4680 1701 50  0000 L CNN
-F 2 "Connector_JST:JST_PH_S4B-PH-K_1x04_P2.00mm_Horizontal" H 4600 1800 50  0001 C CNN
-F 3 "~" H 4600 1800 50  0001 C CNN
-	1    4600 1800
-	-1   0    0    1
+P 4600 1700
+F 0 "J2" H 4680 1692 50  0000 L CNN
+F 1 "Conn_01x04" H 4680 1601 50  0000 L CNN
+F 2 "Connector_JST:JST_PH_S4B-PH-K_1x04_P2.00mm_Horizontal" H 4600 1700 50  0001 C CNN
+F 3 "~" H 4600 1700 50  0001 C CNN
+	1    4600 1700
+	-1   0    0    -1
 $EndComp
 $Comp
@@
 	6200 4500 7000 4500
 Connection ~ 6200 4500
-$Comp
-L driver-rescue:VXO7805-500-M-VXO7805-500-M PS1
-U 1 1 60157AFB
-P 6200 4000
-F 0 "PS1" H 6200 4467 50  0000 C CNN
-F 1 "VXO7805-500-M" H 6200 4376 50  0000 C CNN
-F 2 "CONV_VXO7805-500-M" H 6200 4000 50  0001 L BNN
-F 3 "" H 6200 4000 50  0001 L BNN
-F 4 "1.0" H 6200 4000 50  0001 L BNN "PARTREV"
-F 5 "CUI Inc." H 6200 4000 50  0001 L BNN "MANUFACTURER"
-F 6 "3.5 mm" H 6200 4000 50  0001 L BNN "MAXIMUM_PACKAGE_HEIGHT"
-F 7 "Manufacturer Recommendations" H 6200 4000 50  0001 L BNN "STANDARD"
-	1    6200 4000
-	1    0    0    -1
-$EndComp
 Wire Wire Line
 	4850 4500 5200 4500
 Connection ~ 5200 4500
 Wire Wire Line
-	5200 4500 6200 4500
+	5200 4500 5500 4500
 Wire Wire Line
 	5200 4200 5200 3800
@@
 	1    0    0    -1
 $EndComp
+$Comp
+L VXO7805-500-M:VXO7805-500-M PS1
+U 1 1 6042EFCA
+P 6200 4000
+F 0 "PS1" H 6200 4467 50  0000 C CNN
+F 1 "VXO7805-500-M" H 6200 4376 50  0000 C CNN
+F 2 "CONV_VXO7805-500-M" H 6200 4000 50  0001 L BNN
+F 3 "1.0" H 6200 4000 50  0001 L BNN
+F 4 "3.5 mm" H 6200 4000 50  0001 L BNN "Field4"
+F 5 "CUI Inc." H 6200 4000 50  0001 L BNN "Field5"
+F 6 "Manufacturer Recommendations" H 6200 4000 50  0001 L BNN "Field6"
+	1    6200 4000
+	1    0    0    -1
+$EndComp
+Wire Wire Line
+	5500 4200 5500 4500
+Connection ~ 5500 4500
+Wire Wire Line
+	5500 4500 6200 4500
 $EndSCHEMATC
