File: analog-driver/driver.kicad_pcb (KiCad board)
At the start: 2 copper layers, 81 x 23.4 mm, 18 parts, among them J1 Conn_01x02, J2 Barrel_Jack, J3 Barrel_Jack, M1 Fan_4pin, U1 AL8805W5-7, U2 LM2941S

Commit message: analog driver 1.0.0
Parts:
- removed C1: 1uF, Capacitor_SMD:C_1206_3216Metric
- removed C3: 0.47uF, Capacitor_SMD:C_1206_3216Metric
- removed C4: 22uF, Capacitor_SMD:C_1206_3216Metric
- removed J1: Conn_01x02, Connector_PinSocket_2.54mm:PinSocket_1x02_P2.54mm_Vertical
- removed J2: Barrel_Jack, Connector_BarrelJack:BarrelJack_Horizontal
- removed L1: 33uH, Inductor_SMD:L_Bourns_SRR1260
- removed M1: Fan_4pin, Connector:FanPinHeader_1x04_P2.54mm_Vertical
- removed the REF** at (110.7, 128.0)
- removed the REF** at (184.5, 128.3)
- removed RV2: 5kOhm1, Potentiometer_THT:Potentiometer_Bourns_3296Y_Vertical
- removed U1: AL8805W5-7, AL8805W5-7:SOT95P280X130-5N
- added G***: LOGO, footprints:logo, F.Cu at (127.0, 95.2)
- added J4: Barrel_Jack, Connector_BarrelJack:BarrelJack_Horizontal, F.Cu at (95.2, 101.6)
- added J5: Conn_01x04, Connector_PinHeader_2.54mm:PinHeader_1x04_P2.54mm_Vertical, F.Cu at (146.1, 106.7)
- added J7: Conn_01x02, Connector_PinSocket_2.54mm:PinSocket_1x02_P2.54mm_Vertical, F.Cu at (113.0, 82.5)
- added R5: 1k, Resistor_SMD:R_1206_3216Metric_Pad1.30x1.75mm_HandSolder, F.Cu at (135.9, 94.0)
- added REF**: MountingHole_3.7mm, MountingHole:MountingHole_3.7mm, F.Cu at (152.4, 101.6)
- added REF**: MountingHole_3.7mm, MountingHole:MountingHole_3.7mm, F.Cu at (101.6, 101.6)
- added TP1: TestPoint, TestPoint:TestPoint_THTPad_D3.0mm_Drill1.5mm, F.Cu at (89.5, 82.5)
- added TP2: TestPoint, TestPoint:TestPoint_THTPad_D3.0mm_Drill1.5mm, F.Cu at (164.5, 88.9)
- added TP3: TestPoint, TestPoint:TestPoint_THTPad_D3.0mm_Drill1.5mm, F.Cu at (164.5, 82.5)
- C2: value 2.2uF -> 10u; footprint Capacitor_SMD:C_1206_3216Metric -> Capacitor_SMD:C_1206_3216Metric_Pad1.33x1.80mm_HandSolder
- D1: value MBRA140 -> LED; footprint MBRA140:SMA-DIODE -> LED_SMD:LED_1206_3216Metric
- R1: value 0.3R -> 10k; footprint Resistor_SMD:R_1206_3216Metric -> Resistor_SMD:R_1206_3216Metric_Pad1.30x1.75mm_HandSolder
- R2: value 8KOhm -> 470; footprint Resistor_SMD:R_1206_3216Metric -> Resistor_SMD:R_1206_3216Metric_Pad1.30x1.75mm_HandSolder
- RV1: value 100KOhm -> 2.2k; footprint Potentiometer_THT:Potentiometer_Bourns_3296Y_Vertical -> footprints:TRIM_3362P-1-202TLF
- U2: value LM2941S -> LDD-1500L; footprint LM2941S:VREG_TPS79625KTTR -> LDD-1500L:LDD1500L; moved to B.Cu
- moved R2 68.7 mm to (92.7, 93.3), turned to 270 degrees
- moved R1 64.3 mm to (97.8, 93.3), turned to 90 degrees
- moved RV1 57.9 mm to (97.8, 86.4), turned to 0 degrees
- moved D1 27.3 mm to (135.9, 99.1), turned to 0 degrees
- moved C2 26.9 mm to (148.6, 88.0)
- moved J3 23.7 mm to (158.8, 101.6)
- moved U2 21.1 mm to (141.0, 104.8), turned to 90 degrees
Connections:
- R1 pad 1: Net-(C1-Pad1) -> +12V
- R1 pad 2: +12V -> Net-(R1-Pad2)
- R2 pad 1: Net-(C4-Pad1) -> Net-(R2-Pad1)
- R2 pad 2: Net-(R2-Pad2) -> GND
- RV1 pad 1: +12V -> Net-(R2-Pad1)
- RV1 pad 2: Net-(RV1-Pad2) -> Net-(R1-Pad2)
- RV1 pad 3: GND -> Net-(R1-Pad2)
- U2 pad 1: Net-(RV2-Pad2) -> GND
Routing:
- net GND: track 217.1 -> 0.00 mm
- net Net-(R1-Pad2): track 0.00 -> 54.7 mm
- net +12V: track 168.8 -> 126.1 mm
- net Net-(C4-Pad1): track 38.4 -> 0.00 mm
- net Net-(C1-Pad1): track 29.5 -> 0.00 mm
- net Net-(RV2-Pad2): track 28.3 -> 0.00 mm
- net Net-(J7-Pad2): track 0.00 -> 26.9 mm
- net Net-(RV1-Pad2): track 25.5 -> 0.00 mm
- net Net-(C1-Pad2): track 16.7 -> 0.00 mm
- net Net-(D1-PadA): track 16.7 -> 0.00 mm
- net Net-(J7-Pad1): track 0.00 -> 9.52 mm
- net Net-(R2-Pad1): track 0.00 -> 6.49 mm
- net Net-(D1-Pad2): track 0.00 -> 5.14 mm
- net Net-(R2-Pad2): track 4.70 -> 0.00 mm
- added copper zone on B.Cu, net GND
- added copper zone on F.Cu, net GND
Other:
- board size 81 x 23.4 mm -> 81.3 x 30.5 mm
- net class Default: clearance 0.2 -> 0.381; trace_width 0.25 -> 0.889
- rule trace_clearance: 0.2 -> 0.381
- board text added: "12 V DC CENTER POSITIVE"
- board text added: "DIM"
- board text added: "DIM 0 to 2.5 V 0 to 100 %"
- board text added: "FAN"
- board text added: "GND"
- board text added: "LED"
- board text added: "PHOTOREACTOR DRIVER"
- board text added: "POWER"
- board text added: "REVISION 1.0.0 JANUARY 2021"
- board text added: "V+"
- board text removed: "Analog Photoreactor Controller"
- board text removed: "FAN PLUG"
- board text removed: "FAN POT"
- board text removed: "Gellman Group"
- board text removed: "LED PLUG"
- board text removed: "LED POT"
- board text removed: "Nov 2020"
- board text removed: "Philip Lampkin"
- board text removed: "V1.0"

Commit message: analog-driver revision B
Parts:
- R1: value 10k -> 6.8k
- R2: value 470 -> 100
- moved C2 0.34 mm to (148.6, 87.6)
Connections:
- J5 pad 3: Net-(J5-Pad3) -> (no net)
- J5 pad 4: Net-(J5-Pad4) -> (no net)
Other:
- board text added: "100"
- board text added: "10μF"
- board text added: "1K"
- board text added: "6.8K"
- board text added: "BLAISE THOMPSON UW-MADSION"
- board text added: "BLK"
- board text added: "BLU"
- board text added: "DIM 0.5 to 2.5 V 20 to 100 %"
- board text added: "REVISION B MARCH 2021"
- board text removed: "DIM 0 to 2.5 V 0 to 100 %"
- board text removed: "REVISION 1.0.0 JANUARY 2021"
Changed lines of the file:
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@@
   (general
     (thickness 1.6)
-    (drawings 27)
+    (drawings 33)
     (tracks 39)
     (zones 0)
     (modules 17)
-    (nets 10)
+    (nets 8)
   )
   (page USLetter)
   (title_block
     (title "Digital Photoreactor Driver")
-    (date 2021-01-29)
-    (rev 1.0.0)
+    (date 2021-03-05)
+    (rev B)
     (company "University of Wisconsin-Madison")
     (comment 1 "Department of Chemistry")
@@
   (net 6 "Net-(R2-Pad1)")
   (net 7 "Net-(R1-Pad2)")
-  (net 8 "Net-(J5-Pad4)")
-  (net 9 "Net-(J5-Pad3)")
   (net_class Default "This is the default net class."
     (clearance 0.381)
@@
     (add_net GND)
     (add_net "Net-(D1-Pad2)")
-    (add_net "Net-(J5-Pad3)")
-    (add_net "Net-(J5-Pad4)")
     (add_net "Net-(J7-Pad1)")
     (add_net "Net-(J7-Pad2)")
@@
     (tags "resistor handsolder")
     (attr smd)
-    (fp_text reference R2 (at 0 -1.905 90) (layer F.SilkS)
-      (effects (font (size 1 1) (thickness 0.15)))
-    )
-    (fp_text value 470 (at 0 1.82 90) (layer F.Fab)
+    (fp_text reference R2 (at 1.27 -1.905 90) (layer F.SilkS) hide
+      (effects (font (size 1 1) (thickness 0.15)))
+    )
+    (fp_text value 100 (at 0 1.82 90) (layer F.Fab)
       (effects (font (size 1 1) (thickness 0.15)))
     )
@@
       (effects (font (size 0.8 0.8) (thickness 0.12)))
     )
-    (pad 2 smd roundrect (at 1.55 0 270) (size 1.3 1.75) (layers F.Cu F.Paste F.Mask) (roundrect_rratio 0.1923076923076923)
+    (pad 2 smd roundrect (at 1.55 0 270) (size 1.3 1.75) (layers F.Cu F.Paste F.Mask) (roundrect_rratio 0.1923069230769231)
       (net 1 GND))
-    (pad 1 smd roundrect (at -1.55 0 270) (size 1.3 1.75) (layers F.Cu F.Paste F.Mask) (roundrect_rratio 0.1923076923076923)
+    (pad 1 smd roundrect (at -1.55 0 270) (size 1.3 1.75) (layers F.Cu F.Paste F.Mask) (roundrect_rratio 0.1923069230769231)
       (net 6 "Net-(R2-Pad1)"))
     (model ${KISYS3DMOD}/Resistor_SMD.3dshapes/R_1206_3216Metric.wrl
@@
     (tags "resistor handsolder")
     (attr smd)
-    (fp_text reference R1 (at 0 1.905 90) (layer F.SilkS)
-      (effects (font (size 1 1) (thickness 0.15)))
-    )
-    (fp_text value 10k (at 0 1.82 90) (layer F.Fab)
+    (fp_text reference R1 (at -1.27 1.905 90) (layer F.SilkS) hide
+      (effects (font (size 1 1) (thickness 0.15)))
+    )
+    (fp_text value 6.8k (at 0 1.82 90) (layer F.Fab)
       (effects (font (size 1 1) (thickness 0.15)))
     )
@@
       (effects (font (size 0.8 0.8) (thickness 0.12)))
     )
-    (pad 2 smd roundrect (at 1.55 0 90) (size 1.3 1.75) (layers F.Cu F.Paste F.Mask) (roundrect_rratio 0.1923076923076923)
+    (pad 2 smd roundrect (at 1.55 0 90) (size 1.3 1.75) (layers F.Cu F.Paste F.Mask) (roundrect_rratio 0.1923069230769231)
       (net 7 "Net-(R1-Pad2)"))
-    (pad 1 smd roundrect (at -1.55 0 90) (size 1.3 1.75) (layers F.Cu F.Paste F.Mask) (roundrect_rratio 0.1923076923076923)
+    (pad 1 smd roundrect (at -1.55 0 90) (size 1.3 1.75) (layers F.Cu F.Paste F.Mask) (roundrect_rratio 0.1923069230769231)
       (net 2 +12V))
     (model ${KISYS3DMOD}/Resistor_SMD.3dshapes/R_1206_3216Metric.wrl
@@
   )
   (module Capacitor_SMD:C_1206_3216Metric_Pad1.33x1.80mm_HandSolder (layer F.Cu)
-    (at 148.59 87.9725 270)
+    (at 148.59 87.63 270)
     (descr "Capacitor SMD 1206 (3216 Metric), square (rectangular) end terminal, IPC_7351 nominal with elongated pad for handsoldering. (Body size source: IPC-SM-782 page 76, https://www.pcb-3d.com/wordpress/wp-content/uploads/ipc-sm-782a_amendment_1_and_2.pdf), generated with kicad-footprint-generator")
     (tags "capacitor handsolder")
     (attr smd)
-    (fp_text reference C2 (at 0 -1.85 90) (layer F.SilkS)
+    (fp_text reference C2 (at 0 -1.85 90) (layer F.SilkS) hide
       (effects (font (size 1 1) (thickness 0.15)))
     )
@@
       (effects (font (size 0.8 0.8) (thickness 0.12)))
     )
-    (pad 1 smd roundrect (at -1.5625 0 270) (size 1.325 1.8) (layers F.Cu F.Paste F.Mask) (roundrect_rratio 0.1886784905660377)
+    (pad 1 smd roundrect (at -1.5625 0 270) (size 1.325 1.8) (layers F.Cu F.Paste F.Mask) (roundrect_rratio 0.1886777358490566)
       (net 1 GND))
-    (pad 2 smd roundrect (at 1.5625 0 270) (size 1.325 1.8) (layers F.Cu F.Paste F.Mask) (roundrect_rratio 0.1886784905660377)
+    (pad 2 smd roundrect (at 1.5625 0 270) (size 1.325 1.8) (layers F.Cu F.Paste F.Mask) (roundrect_rratio 0.1886777358490566)
       (net 2 +12V))
     (model ${KISYS3DMOD}/Capacitor_SMD.3dshapes/C_1206_3216Metric.wrl
@@
   (module footprints:TRIM_3362P-1-202TLF (layer F.Cu)
     (at 97.79 86.36)
-    (fp_text reference RV1 (at 0 0.635) (layer F.SilkS)
+    (fp_text reference RV1 (at 0 0.635) (layer F.SilkS) hide
       (effects (font (size 1.002756 1.002756) (thickness 0.015)))
     )
@@
     (tags "resistor handsolder")
     (attr smd)
-    (fp_text reference R5 (at 0 -1.905) (layer F.SilkS)
+    (fp_text reference R5 (at 0 -1.905) (layer F.SilkS) hide
       (effects (font (size 1 1) (thickness 0.15)))
     )
@@
       (effects (font (size 1 1) (thickness 0.15)))
     )
-    (pad 4 thru_hole oval (at 0 7.62 180) (size 1.7 1.7) (drill 1) (layers *.Cu *.Mask)
-      (net 8 "Net-(J5-Pad4)"))
-    (pad 3 thru_hole oval (at 0 5.08 180) (size 1.7 1.7) (drill 1) (layers *.Cu *.Mask)
-      (net 9 "Net-(J5-Pad3)"))
+    (pad 4 thru_hole oval (at 0 7.62 180) (size 1.7 1.7) (drill 1) (layers *.Cu *.Mask))
+    (pad 3 thru_hole oval (at 0 5.08 180) (size 1.7 1.7) (drill 1) (layers *.Cu *.Mask))
     (pad 2 thru_hole oval (at 0 2.54 180) (size 1.7 1.7) (drill 1) (layers *.Cu *.Mask)
       (net 2 +12V))
@@
     )
   )
-  (gr_text "DIM\n0 to 2.5 V\n0 to 100 %" (at 89.535 88.9 270) (layer F.SilkS)
+  (gr_text 10μF (at 150.495 87.63 90) (layer F.SilkS)
+    (effects (font (size 1 1) (thickness 0.15875)))
+  )
+  (gr_text 1K (at 135.89 92.075) (layer F.SilkS)
+    (effects (font (size 1 1) (thickness 0.15875)))
+  )
+  (gr_text 6.8K (at 99.695 93.345 90) (layer F.SilkS)
+    (effects (font (size 1 1) (thickness 0.15875)))
+  )
+  (gr_text 100 (at 94.615 93.345 90) (layer F.SilkS)
+    (effects (font (size 1 1) (thickness 0.15875)))
+  )
+  (gr_text BLU (at 148.59 99.06 90) (layer F.SilkS)
+    (effects (font (size 1 1) (thickness 0.15)))
+  )
+  (gr_text "BLAISE THOMPSON\nUW-MADSION" (at 148.59 82.55) (layer B.SilkS)
+    (effects (font (size 1 1) (thickness 0.25)) (justify mirror))
+  )
+  (gr_text "DIM\n0.5 to 2.5 V\n20 to 100 %" (at 89.535 89.535 270) (layer F.SilkS)
     (effects (font (size 1 1) (thickness 0.15)))
   )
@@
     (effects (font (size 1 1) (thickness 0.15)))
   )
-  (gr_text GND (at 148.59 106.68 90) (layer F.SilkS)
+  (gr_text BLK (at 148.59 106.68 90) (layer F.SilkS)
     (effects (font (size 1 1) (thickness 0.15)))
   )
-  (gr_text - (at 113.03 85.09) (layer F.SilkS)
+  (gr_text + (at 113.03 85.09) (layer F.SilkS)
     (effects (font (size 1 1) (thickness 0.15)))
   )
-  (gr_text + (at 115.57 85.09) (layer F.SilkS)
+  (gr_text - (at 115.57 85.09) (layer F.SilkS)
     (effects (font (size 1 1) (thickness 0.15)))
   )
@@
   (gr_arc (start 165.1 106.68) (end 165.1 109.22) (angle -90) (layer Edge.Cuts) (width 0.1))
   (gr_arc (start 165.1 81.28) (end 167.64 81.28) (angle -90) (layer Edge.Cuts) (width 0.1))
-  (gr_text "REVISION 1.0.0\nJANUARY 2021" (at 142.24 82.55) (layer B.SilkS)
-    (effects (font (size 1 1) (thickness 0.25)) (justify mirror))
+  (gr_text "REVISION B\nMARCH 2021" (at 148.59 82.55) (layer F.SilkS)
+    (effects (font (size 1 1) (thickness 0.25)))
   )
   (segment (start 158.75 101.6) (end 158.75 102.87) (width 0.889) (layer F.Cu) (net 2))
