File: analog-driver/driver.sch (KiCad schematic (older format))
At the start: 16 parts, among them J1 Conn_01x02, J2 Barrel_Jack, J3 Barrel_Jack, M1 Fan_4pin, U1 AL8805W5-7, U2 LM2941S

Commit message: analog driver 1.0.0
Parts:
- removed C1: 1uF, Capacitor_SMD:C_1206_3216Metric, symbol Device:C
- removed C3: 0.47uF, Capacitor_SMD:C_1206_3216Metric, symbol Device:C
- removed C4: 22uF, Capacitor_SMD:C_1206_3216Metric, symbol Device:C
- removed D1: MBRA140, MBRA140:SMA-DIODE, symbol MBRA140:MBRA140
- removed J3: Barrel_Jack, Connector_BarrelJack:BarrelJack_Horizontal, symbol Connector:Barrel_Jack
- removed L1: 33uH, Inductor_SMD:L_Bourns_SRR1260, symbol Device:L
- removed M1: Fan_4pin, Connector:FanPinHeader_1x04_P2.54mm_Vertical, symbol Motor:Fan_4pin
- removed R1: 0.3R, Resistor_SMD:R_1206_3216Metric, symbol Device:R
- removed R2: 8KOhm, Resistor_SMD:R_1206_3216Metric, symbol Device:R
- removed RV1: 100KOhm, Potentiometer_THT:Potentiometer_Bourns_3296Y_Vertical, symbol Device:R_POT_TRIM
- removed RV2: 5kOhm1, Potentiometer_THT:Potentiometer_Bourns_3296Y_Vertical, symbol Device:R_POT_TRIM
- removed U1: AL8805W5-7, AL8805W5-7:SOT95P280X130-5N, symbol AL8805W5-7:AL8805W5-7
- removed U2: LM2941S, LM2941S:VREG_TPS79625KTTR, symbol LM2941S:LM2941S
- added D1: LED, LED_SMD:LED_1206_3216Metric, symbol Device:LED
- added J4: Barrel_Jack, Connector_BarrelJack:BarrelJack_Horizontal, symbol Connector:Barrel_Jack
- added J5: Conn_01x04, Connector_PinHeader_2.54mm:PinHeader_1x04_P2.54mm_Vertical, symbol Connector_Generic:Conn_01x04
- added R1: 10k, Resistor_SMD:R_1206_3216Metric_Pad1.30x1.75mm_HandSolder, symbol Device:R_US
- added R2: 470, Resistor_SMD:R_1206_3216Metric_Pad1.30x1.75mm_HandSolder, symbol Device:R_US
- added R5: 1k, Resistor_SMD:R_1206_3216Metric_Pad1.30x1.75mm_HandSolder, symbol Device:R_US
- added RV1: 2.2k, footprints:TRIM_3362P-1-202TLF, symbol Device:R_POT_US
- added TP1, TP2, TP3: TestPoint, TestPoint:TestPoint_THTPad_D3.0mm_Drill1.5mm, symbol Connector:TestPoint
- added U2: LDD-1500L, LDD-1500L:LDD1500L, symbol LDD-1500L:LDD-1500L
- C2: value 2.2uF -> 10u; footprint Capacitor_SMD:C_1206_3216Metric -> Capacitor_SMD:C_1206_3216Metric_Pad1.33x1.80mm_HandSolder
- renumbered J2 to J3, J1 to J7
Connections:
- net +12V: now also J4.1, J5.2 (Pin_2), R1.1, R5.1, TP2.1, U2.23 (+VIN_1), U2.24 (+VIN_2)
- net GND: now also D1.1 (K), J4.2, J5.1 (Pin_1), R2.2, TP3.1, U2.1 (-VIN_1), U2.2 (-VIN_2)
- net at J7.1 (Pin_1): now also U2.13 (+VOUT_1), U2.14 (+VOUT_2)
- net at J7.2 (Pin_2): now also U2.11 (-VOUT_1), U2.12 (-VOUT_2)
- new net: R1.2, RV1.2, RV1.3, TP1.1, U2.21 (PWM_+ANALOG_DIM)
- new net: R2.1, RV1.1
- new net: D1.2 (A), R5.2
Other:
- note added: "CONTROL RANGE\n0.5 to 2.5 V DC"
- note added: "FAN"
- note added: "LED DRIVER"
- note added: "NF-A12x15 PWM\n130 mA @ 12 V POWER\nPWM 0-5 V"
- note added: "POWER"
- note added: "POWER\nINDICATOR"
- note added: "TWO BARREL JACKS\nFOR DAISY CHAINING"
- note removed: "0.3R = max current of 333 mA"
- note removed: "Analog Control Fan"
- note removed: "Analog Control LED Driver"
- note removed: "Board Power"
- note removed: "Daisy Chain Power"
- note removed: "I’ve added a trim pot to control the driver. It should output constant 330 mA to LEDs."
- note removed: "LM2941S regulates output and allows for trim pot to control Fan speed without using PWM signal."
- note removed: "This LED driver is adapted from SparkFun femtobuck design."
- moved on the sheet: J3, J7

Commit message: analog-driver revision B
Parts:
- R1: value 10k -> 6.8k
- R2: value 470 -> 100
Changed lines of the file:
@@
 Sheet 1 1
 Title "Analog Photoreactor Driver"
-Date "2021-01-29"
-Rev "1.0.0"
+Date "2021-03-05"
+Rev "B"
 Comp "University of Wisconsin-Madison"
 Comment1 "Department of Chemistry"
@@
 P 4400 2050
 F 0 "R2" H 4468 2096 50  0000 L CNN
-F 1 "470" H 4468 2005 50  0000 L CNN
+F 1 "100" H 4468 2005 50  0000 L CNN
 F 2 "Resistor_SMD:R_1206_3216Metric_Pad1.30x1.75mm_HandSolder" V 4440 2040 50  0001 C CNN
 F 3 "~" H 4400 2050 50  0001 C CNN
@@
 P 4400 1450
 F 0 "R1" H 4468 1496 50  0000 L CNN
-F 1 "10k" H 4468 1405 50  0000 L CNN
+F 1 "6.8k" H 4468 1405 50  0000 L CNN
 F 2 "Resistor_SMD:R_1206_3216Metric_Pad1.30x1.75mm_HandSolder" V 4440 1440 50  0001 C CNN
 F 3 "~" H 4400 1450 50  0001 C CNN
