File: digital-driver-board/kicad/driver.kicad_pcb (KiCad board)
At the start: 2 copper layers, 81.3 x 30.5 mm, 23 parts, among them J1 Conn_01x04, J2 Conn_01x04, J3 Barrel_Jack, J4 Barrel_Jack, J5 Conn_01x04, J7 Conn_01x02, U1 ATtiny85-20PU, U2 LDD-1500L

Commit message: remove wisconsin crest logo
Parts:
- removed G***: LOGO, footprints:logo
